File: eagle/ECE110_final/ecu_sch.sch (EAGLE design)
At the start: 1 part, among them IC1 MEGA8-AI

Commit message: ECU Schematics: v1
Parts:
- removed IC1: MEGA8-AI, atmel:MEGA8-AI
- added C1: 0.1uF, SparkFun-Capacitors:0.1UF-25V(+80/-20%)(0603)
- added CDS: M02JST-PTH-2, SparkFun-Connectors:M02JST-PTH-2
- added D1: STATUS, SparkFun-LED:LED-WHITE
- added GATE1, GATE2, IR: (no value), SparkFun-Connectors:M03JST-PTH
- added MOTOR, SPI: (no value), SparkFun-Connectors:M04JST-PTH
- added R1: PHOTOCELLPTH, SparkFun-Sensors:PHOTOCELLPTH
- added R2, R3: 0.3, SparkFun-Resistors:0.3OHM-1/8W-1%(0805)
- added S1: RESET, SparkFun-Electromechanical:SWITCH-MOMENTARY-2-CLOSED
- added U1: L293D, SparkFun-PowerIC:L298
- added U2: ATMEGA328P, SparkFun-DigitalIC:ATMEGA328_SMT
Connections:
- new net GND: C1.2, CDS.2, GATE1.2, GATE2.2, IR.2, R1.P$1, R3.1, S1.1, U1.GND, U2.AGND, U2.GND@1
- new net N$1: U1.IN1, U2.PD5(T1)
- new net N$10: SPI.3, U2.PB3(MOSI/OC2)
- new net N$11: SPI.2, U2.PB4(MISO)
- new net N$12: SPI.1, U2.PB5(SCK)
- new net N$13: GATE1.3, U2.PD2(INT0)
- new net N$14: GATE2.3, U2.PD3(INT1)
- new net N$15: IR.3, U2.PD4(XCK/T0)
- new net N$16: CDS.1, R1.P$2, R2.1, U2.PC0(ADC0)
- new net N$17: S1.2, U2.PC6(/RESET)
- new net N$18: D1.C, R3.2
- new net N$19: D1.A, U2.PB1(OC1A)
- new net N$2: U1.IN3, U2.PD6(AIN0)
- new net N$3: U1.IN2, U2.PB6(XTAL1/TOSC1)
- new net N$4: U1.IN4, U2.PB7(XTAL2/TOSC2)
- new net N$5: MOTOR.1, U1.OUT1
- new net N$6: MOTOR.2, U1.OUT2
- new net N$7: MOTOR.3, U1.OUT3
- new net N$8: MOTOR.4, U1.OUT4
- new net N$9: SPI.4, U2.PB2(SS/OC1B)
- new net VCC: C1.1, GATE1.1, GATE2.1, IR.1, R2.2, U1.ENA, U1.ENB, U1.VLS, U1.VS, U2.VCC@2

Commit message: [Schematics] Complete
Parts:
- added C2: 2.2uF, SparkFun-Capacitors:47UF-10V-10%(TANT)
Connections:
- net GND: now also C2.-
- net VCC: now also C2.+
Other:
- note added: "Bus Decoupler Reduce Ripple"
- moved on the sheet: MOTOR, SPI
Changed lines of the file:
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@@
 <part name="D1" library="SparkFun-LED" deviceset="LED-WHITE" device="" value="STATUS"/>
 <part name="R3" library="SparkFun-Resistors" deviceset="0.3OHM-1/8W-1%(0805)" device="" value="0.3"/>
+<part name="C2" library="SparkFun-Capacitors" deviceset="47UF-10V-10%(TANT)" device="" value="2.2uF"/>
+<part name="SUPPLY5" library="SparkFun-Aesthetics" deviceset="VCC" device=""/>
+<part name="GND5" library="SparkFun-Aesthetics" deviceset="GND" device=""/>
 </parts>
 <sheets>
 <sheet>
 <plain>
+<frame x1="20.32" y1="76.2" x2="78.74" y2="109.22" columns="8" rows="5" layer="91"/>
+<text x="27.94" y="91.44" size="1.778" layer="91">Bus Decoupler
+Reduce Ripple</text>
 </plain>
 <instances>
@@
 <instance part="C1" gate="G$1" x="15.24" y="35.56"/>
 <instance part="U2" gate="G$1" x="60.96" y="40.64"/>
-<instance part="MOTOR" gate="G$1" x="187.96" y="38.1" rot="R180"/>
-<instance part="SPI" gate="G$1" x="187.96" y="15.24" rot="R180"/>
+<instance part="MOTOR" gate="G$1" x="175.26" y="38.1" rot="R180"/>
+<instance part="SPI" gate="G$1" x="129.54" y="15.24" rot="R180"/>
 <instance part="SUPPLY2" gate="G$1" x="119.38" y="55.88"/>
 <instance part="GND2" gate="1" x="124.46" y="30.48"/>
@@
 <instance part="D1" gate="G$1" x="88.9" y="-7.62" rot="R270"/>
 <instance part="R3" gate="G$1" x="78.74" y="-7.62"/>
+<instance part="C2" gate="G$1" x="58.42" y="93.98"/>
+<instance part="SUPPLY5" gate="G$1" x="58.42" y="96.52"/>
+<instance part="GND5" gate="1" x="58.42" y="86.36"/>
 </instances>
 <busses>
@@
 <junction x="165.1" y="58.42"/>
 </segment>
+<segment>
+<pinref part="C2" gate="G$1" pin="-"/>
+<pinref part="GND5" gate="1" pin="GND"/>
+</segment>
 </net>
 <net name="VCC" class="0">
@@
 <pinref part="SUPPLY4" gate="G$1" pin="VCC"/>
 </segment>
+<segment>
+<pinref part="C2" gate="G$1" pin="+"/>
+<pinref part="SUPPLY5" gate="G$1" pin="VCC"/>
+</segment>
 </net>
 <net name="N$1" class="0">
@@
 <pinref part="U1" gate="G$1" pin="OUT1"/>
 <pinref part="MOTOR" gate="G$1" pin="1"/>
-<wire x1="154.94" y1="40.64" x2="182.88" y2="40.64" width="0.1524" layer="91"/>
+<wire x1="154.94" y1="40.64" x2="170.18" y2="40.64" width="0.1524" layer="91"/>
 </segment>
 </net>
@@
 <pinref part="MOTOR" gate="G$1" pin="2"/>
 <pinref part="U1" gate="G$1" pin="OUT2"/>
-<wire x1="182.88" y1="38.1" x2="154.94" y2="38.1" width="0.1524" layer="91"/>
+<wire x1="170.18" y1="38.1" x2="154.94" y2="38.1" width="0.1524" layer="91"/>
 </segment>
 </net>
@@
 <segment>
 <pinref part="U1" gate="G$1" pin="OUT3"/>
-<wire x1="154.94" y1="35.56" x2="182.88" y2="35.56" width="0.1524" layer="91"/>
+<wire x1="154.94" y1="35.56" x2="170.18" y2="35.56" width="0.1524" layer="91"/>
 <pinref part="MOTOR" gate="G$1" pin="3"/>
 </segment>
@@
 <pinref part="MOTOR" gate="G$1" pin="4"/>
 <pinref part="U1" gate="G$1" pin="OUT4"/>
-<wire x1="182.88" y1="33.02" x2="154.94" y2="33.02" width="0.1524" layer="91"/>
+<wire x1="170.18" y1="33.02" x2="154.94" y2="33.02" width="0.1524" layer="91"/>
 </segment>
 </net>
@@
 <segment>
 <pinref part="SPI" gate="G$1" pin="4"/>
-<wire x1="182.88" y1="10.16" x2="99.06" y2="10.16" width="0.1524" layer="91"/>
+<wire x1="124.46" y1="10.16" x2="99.06" y2="10.16" width="0.1524" layer="91"/>
 <wire x1="99.06" y1="10.16" x2="99.06" y2="15.24" width="0.1524" layer="91"/>
 <pinref part="U2" gate="G$1" pin="PB2(SS/OC1B)"/>
@@
 <pinref part="SPI" gate="G$1" pin="3"/>
 <pinref part="U2" gate="G$1" pin="PB3(MOSI/OC2)"/>
-<wire x1="182.88" y1="12.7" x2="86.36" y2="12.7" width="0.1524" layer="91"/>
+<wire x1="124.46" y1="12.7" x2="86.36" y2="12.7" width="0.1524" layer="91"/>
 </segment>
 </net>
@@
 <segment>
 <pinref part="SPI" gate="G$1" pin="2"/>
-<wire x1="182.88" y1="15.24" x2="101.6" y2="15.24" width="0.1524" layer="91"/>
+<wire x1="124.46" y1="15.24" x2="101.6" y2="15.24" width="0.1524" layer="91"/>
 <wire x1="101.6" y1="15.24" x2="101.6" y2="7.62" width="0.1524" layer="91"/>
 <wire x1="101.6" y1="7.62" x2="96.52" y2="7.62" width="0.1524" layer="91"/>
@@
 <segment>
 <pinref part="SPI" gate="G$1" pin="1"/>
-<wire x1="182.88" y1="17.78" x2="93.98" y2="17.78" width="0.1524" layer="91"/>
+<wire x1="124.46" y1="17.78" x2="93.98" y2="17.78" width="0.1524" layer="91"/>
 <wire x1="93.98" y1="17.78" x2="93.98" y2="7.62" width="0.1524" layer="91"/>
 <pinref part="U2" gate="G$1" pin="PB5(SCK)"/>
@@
 </schematic>
 </drawing>
+<compatibility>
+<note version="6.3" minversion="6.2.2" severity="warning">
+Since Version 6.2.2 text objects can contain more than one line,
+which will not be processed correctly with this version.
+</note>
+</compatibility>
 </eagle>
